Commit message: air_simulator packages

File: air_simulator/urdf/air.urdf (robot description, URDF)
Before this commit: robot air, 8 links, 7 joints
Links:
- link laser_link_0: geometry collision cylinder length=0.18 radius=0.0508; visual mesh filename=package://air_simulator/meshes/s300.obj scale=0.001 0.001 0.001
- link laser_link_1: geometry collision cylinder length=0.18 radius=0.0508; visual mesh filename=package://air_simulator/meshes/s300.obj scale=0.001 0.001 0.001

File: air_simulator/urdf/air.xacro (robot description, xacro)
@@ -227,5 +227,5 @@
       <geometry>
         <!-- <cylinder radius="0.0508" length="0.055"/> -->
-<mesh filename="package://air_description/meshes/s300.obj" scale="0.001 0.001 0.001"/>
+<mesh filename="package://air_simulator/meshes/s300.obj" scale="0.001 0.001 0.001"/>
       </geometry>
         <!-- <material name="yellow"/> -->
@@ -261,5 +261,5 @@
       <geometry>
         <!-- <cylinder radius="0.0508" length="0.055"/> -->
-<mesh filename="package://air_description/meshes/s300.obj" scale="0.001 0.001 0.001"/>
+<mesh filename="package://air_simulator/meshes/s300.obj" scale="0.001 0.001 0.001"/>
       </geometry>
       <!-- <material name="yellow"/> -->

Commit message: sick scanners merger and ros gazebo bridge regulations

File: air_simulator/urdf/air.urdf (robot description, URDF)
Before this commit: robot air, 8 links, 7 joints
Links:
- added link camera_link, mass 0.1; collision box size=.03 .03 .03; visual box size=.03 .03 .03
- added link camera_link_optical
- added link imu_link
- added link laser_merger_link
Joints:
- added joint camera_joint: type fixed, parent base_link, child camera_link, origin xyz=0.225 0 0.075 rpy=0 0 0, axis 0 1 0
- added joint camera_optical_joint: type fixed, parent camera_link, child camera_link_optical, origin xyz=0 0 0 rpy=-1.5707 0 -1.5707
- added joint imu_joint: type fixed, parent base_link, child imu_link, origin xyz=0 0 0 rpy=0 0 0
- added joint laser_merger_joint: type fixed, parent base_link, child laser_merger_link, origin xyz=0 0 0.22 rpy=0 0 0

File: air_simulator/urdf/air.xacro (robot description, xacro)
@@ -122,4 +122,53 @@
     <origin xyz="0.0 0.0 ${wheel_zoff+base_height+battery_height/2.0}" rpy="0 0 0"/>
   </joint>
+  <!-- Camera -->
+<joint type="fixed" name="camera_joint">
+    <origin xyz="0.225 0 0.075" rpy="0 0 0"/>
+    <child link="camera_link"/>
+    <parent link="base_link"/>
+    <axis xyz="0 1 0" />
+  </joint>
+  <link name='camera_link'>
+    <pose>0 0 0 0 0 0</pose>
+    <inertial>
+      <mass value="0.1"/>
+      <origin xyz="0 0 0" rpy="0 0 0"/>
+      <inertia
+          ixx="1e-6" ixy="0" ixz="0"
+          iyy="1e-6" iyz="0"
+          izz="1e-6"
+      />
+    </inertial>
+    <collision name='collision'>
+      <origin xyz="0 0 0" rpy="0 0 0"/>
+      <geometry>
+        <box size=".03 .03 .03"/>
+      </geometry>
+    </collision>
+    <visual name='camera_link_visual'>
+      <origin xyz="0 0 0" rpy="0 0 0"/>
+      <geometry>
+        <box size=".03 .03 .03"/>
+      </geometry>
+    </visual>
+  </link>
+  <gazebo reference="camera_link">
+    <material>Gazebo/Red</material>
+  </gazebo>
+  <joint type="fixed" name="camera_optical_joint">
+    <origin xyz="0 0 0" rpy="-1.5707 0 -1.5707"/>
+    <child link="camera_link_optical"/>
+    <parent link="camera_link"/>
+  </joint>
+  <link name="camera_link_optical">
+  </link>
+  <!-- IMU -->
+  <joint name="imu_joint" type="fixed">
+    <origin xyz="0 0 0" rpy="0 0 0" />
+    <parent link="base_link"/>
+    <child link="imu_link" />
+  </joint>
+  <link name="imu_link">
+  </link>
   <!-- Wheels -->
   <xacro:macro name="wheel" params="prefix x_reflect y_reflect">
